Commit message: make distinction between ignition and gazebo classic for the camera; at the moment it seems, that in both cases only the central rgbd camera is considered and the stereo (depth) camera seems to be missing in both cases

File: turtlebot4_description/urdf/sensors/oakd.urdf.xacro (robot description, xacro)
@@ -3,5 +3,5 @@
 <xacro:macro name="oakd" params="name:=oakd parent_link *origin model:=pro">
   <xacro:include filename="$(find irobot_create_description)/urdf/common_properties.urdf.xacro"/>
-  <xacro:property name="mass"       value="0.061"/>
+  <xacro:property name="mass"     value="0.061"/>
   <xacro:property name="baseline" value="0.075" />
   <xacro:property name="M_PI"     value="3.1415926535897931" />
@@ -98,24 +98,58 @@
   </joint>
   <!-- Gazebo links and joints -->
-  <gazebo reference="${name}_rgb_camera_frame">
-    <sensor name="rgbd_camera" type="rgbd_camera">
-      <camera>
-        <horizontal_fov>1.25</horizontal_fov>
-        <image>
-          <width>320</width>
-          <height>240</height>
-        </image>
-        <clip>
-          <near>0.3</near>
-          <far>100</far>
-        </clip>
-        <optical_frame_id>${name}_rgb_camera_optical_frame</optical_frame_id>
-      </camera>
-      <always_on>1</always_on>
-      <update_rate>30</update_rate>
-      <visualize>true</visualize>
-    </sensor>
-    <xacro:material_darkgray/>
-  </gazebo>
+  <xacro:if value="${'$(arg gazebo)' == 'classic'}">
+    <gazebo reference="${name}_rgb_camera_frame">
+      <sensor name="rgbd_camera" type="camera">
+        <camera>
+          <horizontal_fov>1.25</horizontal_fov>
+          <image>
+            <width>320</width>
+            <height>240</height>
+          </image>
+          <clip>
+            <near>0.3</near>
+            <far>100</far>
+          </clip>
+          <optical_frame_id>${name}_rgb_camera_optical_frame</optical_frame_id>
+        </camera>
+        <always_on>1</always_on>
+        <update_rate>30</update_rate>
+        <visualize>true</visualize>
+        <plugin name="rgbd_camera" filename="libgazebo_ros_camera.so">
+          <ros>
+            <!-- <namespace>test_cam</namespace> -->
+            <remapping>image_raw:=image_demo</remapping>
+            <remapping>camera_info:=camera_info_demo</remapping>
+          </ros>
+          <!-- camera_name>omit so it defaults to sensor name</camera_name-->
+          <!-- frame_name>omit so it defaults to link name</frameName-->
+          <!-- <hack_baseline>0.07</hack_baseline> -->
+        </plugin>
+      </sensor>
+      <xacro:material_darkgray/>
+    </gazebo>
+  </xacro:if>
+  <xacro:if value="${'$(arg gazebo)' == 'ignition'}">
+    <gazebo reference="${name}_rgb_camera_frame">
+      <sensor name="rgbd_camera" type="rgbd_camera">
+        <camera>
+          <horizontal_fov>1.25</horizontal_fov>
+          <image>
+            <width>320</width>
+            <height>240</height>
+          </image>
+          <clip>
+            <near>0.3</near>
+            <far>100</far>
+          </clip>
+          <optical_frame_id>${name}_rgb_camera_optical_frame</optical_frame_id>
+        </camera>
+        <always_on>1</always_on>
+        <update_rate>30</update_rate>
+        <visualize>true</visualize>
+      </sensor>
+      <xacro:material_darkgray/>
+    </gazebo>
+  </xacro:if>
   <gazebo reference="${name}_joint">
     <preserveFixedJoint>true</preserveFixedJoint>
